Commit message: - Modified the camera link location and added the camera optical frame link

File: seekur_jr_description/robots/seekur_jr_with_arm.urdf.xacro (robot description, xacro)
@@ -17,4 +17,13 @@
     <origin xyz="0.3525 0 0"/> <!-- 0.425/2 + ~0.14 -->
   </joint>
+  <property name="cal_xtion_x" value="0.0" />
+  <property name="cal_xtion_y" value="0.0" />
+  <property name="cal_xtion_z" value="0.0" />
+  <property name="cal_xtion_roll" value="0.0" />
+  <property name="cal_xtion_pitch" value="0.0" />
+  <property name="cal_xtion_yaw" value="0.0" />
+  <!-- xacro:xtion_camera_v0 name="camera" parent="arm_base_link" -->
+     <!--origin xyz="0.622392 -0.999073 0.41495" rpy="0.0150779 0.386473 1.57926"/ -->
+  <!-- /xacro:xtion_camera_v0  -->
   <xacro:include filename="$(find seekur_jr_description)/urdf/seekur_jr.xacro" />
   <xacro:include filename="$(find seekur_jr_description)/urdf/sensors/sensors.xacro" />

File: seekur_jr_description/urdf/seekur_jr.xacro (robot description, xacro)
@@ -25,31 +25,5 @@
     </inertial>
   </link>
-  <joint name="camera_joint" type="fixed">
-      <origin xyz="0.53 0 0.36" rpy="0 0 0" /> <!-- 386 + 20 plaque -->
-      <parent link="base_link"/>
-      <child link="camera_link"/>
-  </joint>
-  <link name="camera_link" >
-    <visual>
-      <origin xyz="-0.005 0.09 -0.01" rpy="${pi*0.31} 0 ${-pi/2}" />
-      <geometry>
-        <mesh filename="package://seekur_jr_description/meshes/camera_box.stl" scale="0.001 0.001 0.001"/>
-      </geometry>
-      <material name="Blue"/>
-    </visual>
-      <collision>
-      <origin xyz="0 0 0" rpy="${pi/2} 0 ${-pi/2}" />
-      <geometry>
-        <mesh filename="package://seekur_jr_description/meshes/camera_box.stl" scale="0.001 0.001 0.001"/>
-      </geometry>
-    </collision>
-    <inertial>
-      <mass value="1" />
-      <origin xyz="0 0 0" rpy="0 0 0"/>
-      <inertia ixx="1" ixy="0" ixz="0"
-	       iyy="1" iyz="0"
-               izz="1" />
-    </inertial>
-  </link>
+    <!--  here was the camera link and joint -->
   <joint name="seekur_base_to_top_joint" type="fixed">
       <origin xyz="0 0 0.406" rpy="0 0 0" /> <!-- 386 + 20 plaque -->

File: seekur_jr_description/urdf/sensors/sensors.xacro (robot description, xacro)
@@ -7,4 +7,76 @@
     <origin xyz="0.55 0 0.23"/>
   </joint>
+ <joint name="camera_joint" type="fixed">
+      <origin xyz="0.53 0 0.36" rpy="0 ${pi*0.123} 0" /> <!-- 386 + 20 plaque -->
+      <parent link="base_link"/>
+      <child link="camera_link"/>
+  </joint>
+  <link name="camera_link" >
+    <visual>
+      <origin xyz="0.001 0.09 -0.01" rpy="${pi*0.51} 0 ${-pi/2}" />
+      <geometry>
+        <mesh filename="package://seekur_jr_description/meshes/camera_box.stl" scale="0.001 0.001 0.001"/>
+      </geometry>
+      <material name="Blue"/>
+    </visual>
+      <collision>
+      <origin xyz="0 0 0" rpy="${pi/2} 0 ${-pi/2}" />
+      <geometry>
+        <mesh filename="package://seekur_jr_description/meshes/camera_box.stl" scale="0.001 0.001 0.001"/>
+      </geometry>
+    </collision>
+    <inertial>
+      <mass value="1" />
+      <origin xyz="0 0 0" rpy="0 0 0"/>
+      <inertia ixx="1" ixy="0" ixz="0"
+	       iyy="1" iyz="0"
+               izz="1" />
+    </inertial>
+  </link>
+   <joint name="camera_optical_joint" type="fixed">
+      <origin xyz="${cal_xtion_x}           ${cal_xtion_y}         ${cal_xtion_z}"
+                rpy="${-pi/2+cal_xtion_roll} ${0.0+cal_xtion_pitch} ${-pi/2+cal_xtion_yaw}" />
+      <parent link="camera_link"/>
+      <child link="camera_optical_frame"/>
+    </joint>
+    <link name="camera_optical_frame"/>
+    <!-- not sure of this part ( arm_base_link .. camera calibration ) -->
+   <!--
+      <xacro:macro name="xtion_camera_v0" params="name parent *origin">
+    <joint name="${name}_frame_joint" type="fixed">
+      <insert_block name="origin" />
+      <parent link="${parent}"/>
+      <child link="${name}_link"/>
+    </joint>
+    <link name="${name}_link">
+      <inertial>
+        <mass value="0.1" />
+        <origin xyz="0 0 0" rpy="0 0 0"/>
+        <inertia ixx="0.01"  ixy="0.0"  ixz="0.0"
+                 iyy="0.01"  iyz="0.0"
+                 izz="0.01" />
+      </inertial>
+      <visual>
+	<origin xyz="0.0 0.012 0" rpy="0 0 0"/>
+        <geometry>
+          <mesh filename="package://seekur_jr_description/meshes/camera_box.stl" scale="0.001 0.001 0.001" />
+        </geometry>
+      </visual>
+      <collision>
+        <origin xyz="0.0 0.012 0" rpy="0 0 0"/>
+        <geometry>
+          <mesh filename="package://seekur_jr_description/meshes/camera_box.stl" scale="0.001 0.001 0.001" />
+        </geometry>
+      </collision>
+    </link>
+    <joint name="${name}_optical_joint" type="fixed">
+      <origin xyz="${cal_xtion_x}           ${cal_xtion_y}         ${cal_xtion_z}"
+                rpy="${-M_PI/2+cal_xtion_roll} ${0.0+cal_xtion_pitch} ${-M_PI/2+cal_xtion_yaw}" />
+      <parent link="${name}_link"/>
+      <child link="${name}_optical_frame"/>
+    </joint>
+    <link name="${name}_optical_frame"/>
+  </xacro:macro>
+  -->
   <link name="laser">
   </link>

Commit message: - Modification for testing calibration accuracy

File: seekur_jr_description/robots/seekur_jr_with_arm.urdf.xacro (robot description, xacro)
@@ -23,9 +23,9 @@
   <property name="cal_xtion_pitch" value="0.0" />
   <property name="cal_xtion_yaw" value="0.0" />
-  <!-- xacro:xtion_camera_v0 name="camera" parent="arm_base_link" -->
-     <!--origin xyz="0.622392 -0.999073 0.41495" rpy="0.0150779 0.386473 1.57926"/ -->
-  <!-- /xacro:xtion_camera_v0  -->
   <xacro:include filename="$(find seekur_jr_description)/urdf/seekur_jr.xacro" />
-  <xacro:include filename="$(find seekur_jr_description)/urdf/sensors/sensors.xacro" />
   <xacro:include filename="$(find terabot_description)/urdf/terabot.xacro" />
+  <xacro:include filename="$(find seekur_jr_description)/urdf/sensors/sensors.urdf.xacro" />
+ <!-- <xacro:xtion_camera_v0 name="camera" parent="arm_base_link" >
+     <origin xyz="0.148229 0.0529445 -0.0454258" rpy="-0.0173235 0.407733 -0.016268"/>
+   </xacro:xtion_camera_v0> -->
 </robot>

File: seekur_jr_description/urdf/sensors/sensors.urdf.xacro (robot description, xacro)
@@ -7,7 +7,9 @@
     <origin xyz="0.55 0 0.23"/>
   </joint>
- <joint name="camera_joint" type="fixed">
-      <origin xyz="0.53 0 0.36" rpy="0 ${pi*0.123} 0" /> <!-- 386 + 20 plaque -->
-      <parent link="base_link"/>
+   <link name="laser">
+  </link>
+  <joint name="camera_joint" type="fixed">
+      <origin xyz="0.148229 0.0529445 -0.0454258" rpy="-0.0173235 0.407733 -0.016268" />
+      <parent link="arm_base_link"/>
       <child link="camera_link"/>
   </joint>
@@ -42,6 +44,5 @@
     <link name="camera_optical_frame"/>
     <!-- not sure of this part ( arm_base_link .. camera calibration ) -->
-   <!--
-      <xacro:macro name="xtion_camera_v0" params="name parent *origin">
+  <!--    <xacro:macro name="xtion_camera_v0" params="name parent *origin">
     <joint name="${name}_frame_joint" type="fixed">
       <insert_block name="origin" />
@@ -72,12 +73,9 @@
     <joint name="${name}_optical_joint" type="fixed">
       <origin xyz="${cal_xtion_x}           ${cal_xtion_y}         ${cal_xtion_z}"
-                rpy="${-M_PI/2+cal_xtion_roll} ${0.0+cal_xtion_pitch} ${-M_PI/2+cal_xtion_yaw}" />
+                rpy="${-pi/2+cal_xtion_roll} ${0.0+cal_xtion_pitch} ${-pi/2+cal_xtion_yaw}" />
       <parent link="${name}_link"/>
       <child link="${name}_optical_frame"/>
     </joint>
     <link name="${name}_optical_frame"/>
-  </xacro:macro>
-  -->
-  <link name="laser">
-  </link>
+  </xacro:macro> -->
 </robot>
