Commit message: - Added the xtion camera link/joint and changed the laser sensor joint location

File: seekur_jr_description/urdf/seekur_jr.xacro (robot description, xacro)
@@ -15,4 +15,31 @@
       <geometry>
         <mesh filename="package://seekur_jr_description/meshes/SeekurJr.stl" scale="0.001 0.001 0.001"/>
+      </geometry>
+    </collision>
+    <inertial>
+      <mass value="100" />
+      <origin xyz="0 0 0" rpy="0 0 0"/>
+      <inertia ixx="1" ixy="0" ixz="0"
+	       iyy="1" iyz="0"
+               izz="1" />
+    </inertial>
+  </link>
+  <joint name="camera_xtion_joint" type="fixed">
+      <origin xyz="0.53 0 0.36" rpy="0 0 0" /> <!-- 386 + 20 plaque -->
+      <parent link="base_link"/>
+      <child link="camera_xtion_link"/>
+  </joint>
+  <link name="camera_xtion_link" >
+    <visual>
+      <origin xyz="-0.005 0.09 -0.01" rpy="${pi*0.31} 0 ${-pi/2}" />
+      <geometry>
+        <mesh filename="package://seekur_jr_description/meshes/camera_box.stl" scale="0.001 0.001 0.001"/>
+      </geometry>
+      <material name="Blue"/>
+    </visual>
+      <collision>
+      <origin xyz="0 0 0" rpy="${pi/2} 0 ${-pi/2}" />
+      <geometry>
+        <mesh filename="package://seekur_jr_description/meshes/camera_box.stl" scale="0.001 0.001 0.001"/>
       </geometry>
     </collision>

File: seekur_jr_description/urdf/sensors/sensors.xacro (robot description, xacro)
@@ -5,5 +5,5 @@
     <parent link="base_link"/>
     <child link="laser"/>
-    <origin xyz="0.55 0 0.2"/>
+    <origin xyz="0.55 0 0.23"/>
   </joint>
   <link name="laser">

Commit message: -fixed some color issues

File: seekur_jr_description/urdf/seekur_jr.xacro (robot description, xacro)
@@ -9,5 +9,5 @@
         <mesh filename="package://seekur_jr_description/meshes/SeekurJr.stl" scale="0.001 0.001 0.001"/>
       </geometry>
-      <material name="Gray"/>
+      <material name="Blue"/>
     </visual>
     <collision>

Commit message: - modified urdf file of the seekur jr

File: seekur_jr_description/urdf/seekur_jr.xacro (robot description, xacro)
@@ -25,10 +25,10 @@
     </inertial>
   </link>
-  <joint name="camera_xtion_joint" type="fixed">
+  <joint name="camera_joint" type="fixed">
       <origin xyz="0.53 0 0.36" rpy="0 0 0" /> <!-- 386 + 20 plaque -->
       <parent link="base_link"/>
-      <child link="camera_xtion_link"/>
+      <child link="camera_link"/>
   </joint>
-  <link name="camera_xtion_link" >
+  <link name="camera_link" >
     <visual>
       <origin xyz="-0.005 0.09 -0.01" rpy="${pi*0.31} 0 ${-pi/2}" />

Commit message: - I can replicate the stupid behaviour observed in the real platform on Gazebo

File: seekur_jr_description/urdf/seekur_jr.xacro (robot description, xacro)
@@ -21,11 +21,11 @@
       </geometry>
     </collision>
+    <!-- KDL Does not support root link with inertia: but without it there will be no mass :( we have to cope with the annoying warnings for the time being -->
     <inertial>
       <mass value="100" />
       <origin xyz="0 0 0" rpy="0 0 0"/>
-      <!-- KDL Does not support root link with inertia -->
-      <inertia ixx="1" ixy="0" ixz="0"
-               iyy="1" iyz="0"
-               izz="1" />
+      <inertia ixx="0" ixy="0" ixz="0"
+               iyy="0" iyz="0"
+               izz="0" />
     </inertial>
   </link>

File: seekur_jr_description/urdf/sensors/sensors.xacro (robot description, xacro)
@@ -39,5 +39,5 @@
   -->
   <xtion parent="arm_base_link">
-    <origin xyz="${0.148229 + cal_xtion_x} ${0.0529445 + cal_xtion_y} ${-0.0454258 + cal_xtion_z}" rpy="${-0.0173235 + cal_xtion_roll} ${0.407733 +cal_xtion_pitch} ${-0.016268 + cal_xtion_yaw}" />
+    <origin xyz="${0.148229 + cal_xtion_x} ${0.0529445/2.0 + cal_xtion_y} ${-0.0454258 + cal_xtion_z}" rpy="${-0.0173235 + cal_xtion_roll} ${0.407733 +cal_xtion_pitch} ${-0.016268 + cal_xtion_yaw}" />
   </xtion>
 </robot>
