Commit message: - Finally, a proper urdf model!

File: seekur_jr_description/urdf/seekur_jr_original.xacro (robot description, xacro)
@@ -153,4 +153,9 @@
       <origin xyz="-0.2125 0.30 0.085" rpy="0 0 0" />
       <axis xyz="0 1 0" rpy="0 0 0" />
+  </joint>
+  <joint name="base_to_arm" type="fixed">
+      <parent link="seekur_top_link"/>
+      <child link="arm_base_link"/>
+      <origin xyz="0.3525 0 0"/>
   </joint>
   <!-- Transmission is important to link the joints and the controller -->
@@ -216,9 +221,4 @@
   </joint>
   -->
-  <joint name="base_to_arm" type="fixed">
-    <parent link="seekur_top_link"/>
-    <child link="arm_base_link"/>
-    <origin xyz="0.3525 0 0"/>
-  </joint>
   <link name="arm_base_link">
     <visual>
@@ -231,5 +231,5 @@
     <collision>
        <geometry>
-        <cylinder length="${80*BASE}" radius="${2*link_radius}"/>
+        <cylinder length="${75*BASE}" radius="${2*link_radius}"/>
       </geometry>
       <origin xyz="0 0 ${(229/4)*BASE}"/>
@@ -254,14 +254,14 @@
   <link name="shoulder_link">
     <visual>
-      <origin xyz="0 0 0" rpy="0 ${-pi/2} ${-pi/2}" />
-      <geometry>
-        <mesh filename="package://seekur_jr_description/meshes/arm/shoulder_n.stl" scale="0.001 0.001 0.001"/>
-      </geometry>
-      <material name="orange"/>
-    </visual>
-    <collision>
-      <origin xyz="0 0 0" rpy="0 ${-pi/2} ${-pi/2}" />
-      <geometry>
-        <mesh filename="package://seekur_jr_description/meshes/arm/shoulder_n.stl" scale="0.001 0.001 0.001"/>
+      <origin xyz="0 0 ${-(80/2)*BASE}" rpy="0 ${-pi/2} ${-pi/2}" />
+      <geometry>
+        <mesh filename="package://seekur_jr_description/meshes/arm/shoulder.stl" scale="0.001 0.001 0.001"/>
+      </geometry>
+      <material name="orange"/>
+    </visual>
+    <collision>
+      <origin xyz="0 0 ${-(80/2)*BASE}" rpy="0 ${-pi/2} ${-pi/2}" />
+      <geometry>
+        <mesh filename="package://seekur_jr_description/meshes/arm/shoulder.stl" scale="0.001 0.001 0.001"/>
       </geometry>
       <material name="orange"/>
@@ -277,6 +277,6 @@
   </link>
   <joint name="forearm_joint" type="revolute">
-    <origin xyz="0 ${-40*BASE} ${108*BASE}" rpy="0 0 ${-PI}"/>
-    <axis xyz="0 1 0"/>
+    <origin xyz="0 0 ${(229/2)*BASE}" rpy="${PI/2} ${-PI/2} ${-PI}"/>
+    <axis xyz="0 0 1"/>
     <limit effort="1000.0" lower="${-90*(PI/180)}" upper="${0*(PI/180)}" velocity="0.5"/>
     <parent link="shoulder_link"/>
@@ -286,14 +286,14 @@
   <link name="forearm_link">
     <visual>
-      <origin xyz="0 0 0" rpy="0 0 0" />
-      <geometry>
-        <mesh filename="package://seekur_jr_description/meshes/arm/forearm_n.stl" scale="0.001 0.001 0.001"/>
-      </geometry>
-      <material name="orange"/>
-    </visual>
-    <collision>
-      <origin xyz="0 0 0" rpy="0 0 0" />
-      <geometry>
-        <mesh filename="package://seekur_jr_description/meshes/arm/forearm_n.stl" scale="0.001 0.001 0.001"/>
+      <origin xyz="${-(229/2)*BASE+forearm_link_x_offset} ${-(229/2)*BASE+forearm_link_y_offset} 0" rpy="0 0 ${PI/4}" />
+      <geometry>
+        <mesh filename="package://seekur_jr_description/meshes/arm/forearm.stl" scale="0.001 0.001 0.001"/>
+      </geometry>
+      <material name="orange"/>
+    </visual>
+    <collision>
+      <origin xyz="${-(229/2)*BASE+forearm_link_x_offset} ${-(229/2)*BASE+forearm_link_y_offset} 0" rpy="0 0 ${PI/4}" />
+      <geometry>
+        <mesh filename="package://seekur_jr_description/meshes/arm/forearm.stl" scale="0.001 0.001 0.001"/>
       </geometry>
       <material name="orange"/>
@@ -309,5 +309,5 @@
   </link>
   <joint name="upper_arm_joint" type="revolute">
-    <origin xyz="${419.1*BASE} ${-65*BASE} 0" rpy="${PI/2.0} 0 0"/>
+    <origin xyz="${419.1*BASE} 0 0" rpy="0 0 0"/>
     <axis xyz="0 0 1"/>
     <limit effort="1000.0" lower="${-170*(PI/180)}" upper="${162*(PI/180)}" velocity="0.5"/>
@@ -318,14 +318,14 @@
   <link name="upper_arm_link">
     <visual>
-      <origin xyz="0 0 0" rpy="0 0 0" />
-      <geometry>
-        <mesh filename="package://seekur_jr_description/meshes/arm/upper_arm_n.stl" scale="0.001 0.001 0.001"/>
-      </geometry>
-      <material name="orange"/>
-    </visual>
-    <collision>
-      <origin xyz="0 0 0" rpy="0 0 0" />
-      <geometry>
-        <mesh filename="package://seekur_jr_description/meshes/arm/upper_arm_n.stl" scale="0.001 0.001 0.001"/>
+      <origin xyz="${(229/2)*BASE+upper_arm_link_x_offset} ${-419.1*BASE-(229/2)*BASE+upper_arm_link_y_offset} 0" rpy="0 0 0" />
+      <geometry>
+        <mesh filename="package://seekur_jr_description/meshes/arm/upper_arm.stl" scale="0.001 0.001 0.001"/>
+      </geometry>
+      <material name="orange"/>
+    </visual>
+    <collision>
+      <origin xyz="${(229/2)*BASE+upper_arm_link_x_offset} ${-419.1*BASE-(229/2)*BASE+upper_arm_link_y_offset} 0" rpy="0 0 0" />
+      <geometry>
+        <mesh filename="package://seekur_jr_description/meshes/arm/upper_arm.stl" scale="0.001 0.001 0.001"/>
       </geometry>
     </collision>
@@ -340,5 +340,5 @@
   </link>
   <joint name="wrist_pitch_joint" type="revolute">
-    <origin xyz="${364.49*BASE} ${7*BASE} 0"/>
+    <origin xyz="${364.49*BASE} 0 0"/>
     <axis xyz="0 0 1"/>
     <limit effort="1000.0" lower="${-170*(PI/180)}" upper="${170*(PI/180)}" velocity="0.5"/>
@@ -349,17 +349,16 @@
   <link name="wrist_pitch_link">
     <visual>
-      <origin xyz="0 0 0" rpy="0 0 0" />
-      <geometry>
-        <mesh filename="package://seekur_jr_description/meshes/arm/wrist_pitch_n.stl" scale="0.001 0.001 0.001"/>
-      </geometry>
-      <material name="orange"/>
-    </visual>
-    <collision>
-      <origin xyz="0 0 0" rpy="0 0 0" />
-      <geometry>
-        <mesh filename="package://seekur_jr_description/meshes/arm/wrist_pitch_n.stl" scale="0.001 0.001 0.001"/>
-      </geometry>
-    </collision>
-    <!--
+      <origin xyz="${(364.49/2)*BASE+wrist_pitch_link_x_offset} ${-419.1*BASE-(229/2)*BASE+wrist_pitch_link_y_offset} 0" rpy="0 0 0" />
+      <geometry>
+        <mesh filename="package://seekur_jr_description/meshes/arm/wrist_pitch.stl" scale="0.001 0.001 0.001"/>
+      </geometry>
+      <material name="orange"/>
+    </visual>
+    <collision>
+      <origin xyz="${(364.49/2)*BASE+wrist_pitch_link_x_offset} ${-419.1*BASE-(229/2)*BASE+wrist_pitch_link_y_offset} 0" rpy="0 0 0" />
+      <geometry>
+          <mesh filename="package://seekur_jr_description/meshes/arm/wrist_pitch.stl" scale="0.001 0.001 0.001"/>
+      </geometry>
+    </collision>
      <visual>
       <origin xyz="${(-100.49/2)*BASE+wrist_pitch_link_x_offset} ${230.1*BASE-(229/2)*BASE+wrist_pitch_link_y_offset} 0" rpy="0 ${PI/2} 0" />
@@ -375,5 +374,4 @@
       </geometry>
     </collision>
-    -->
     <inertial>
       <origin xyz="0 0 0" rpy="0 0 0"/>
@@ -385,10 +383,31 @@
     </inertial>
   </link>
-  <!-- wrist_roll_joint can be used for calibration -->
+ <!-- added end effector for calibration -->
+  <joint name="end_effector_joint" type="fixed">
+    <origin xyz="0.09 ${wrist_roll_joint_z_offset} 0" rpy="0 0 0"/>
+    <axis xyz="0 0 1"/>
+    <parent link="wrist_pitch_link"/>
+    <child link="end_effector"/>
+    <dynamics damping="100.0" friction="100.0" />
+  </joint>
+  <!-- end_effector -->
+  <link name="end_effector">
+    <origin xyz="0 0 0" rpy="0 0 0"/>
+      <inertial>
+        <origin xyz="0 0 1" rpy="0 0 0"/>
+        <mass value="0.01"/>
+        <inertia
+        ixx="1.0" ixy="0.0" ixz="0.0"
+        iyy="1.0" iyz="0.0"
+        izz="1.0"/>
+        </inertial>
+  </link>
+  <!-- modified the following part to add end_effector link (marker) for calibration -->
   <joint name="wrist_roll_joint" type="revolute">
-    <origin xyz="0.09 0.035 ${-20.5*BASE}" rpy="${-PI/2.0} 0 0 "/>
-    <axis xyz="1 0 0"/>
+    <!-- origin xyz="${50*BASE+0.013+wrist_roll_joint_x_offset} ${wrist_roll_joint_z_offset} 0" rpy="0 ${PI/2} 0"/ -->
+    <origin xyz="0.07 0 0" rpy="0 ${PI/2} 0"/>
+    <axis xyz="0 0 1"/>
     <limit effort="1000.0" lower="${-170*(PI/180)}" upper="${170*(PI/180)}" velocity="0.5"/>
-    <parent link="wrist_pitch_link"/>
+    <parent link="end_effector"/>
     <child link="wrist_roll_link"/>
     <dynamics damping="0.7"/>
@@ -396,14 +415,14 @@
   <link name="wrist_roll_link">
     <visual>
-      <origin xyz="0 0 0 " rpy="0 0 0" />
-      <geometry>
-        <mesh filename="package://seekur_jr_description/meshes/arm/wrist_roll_n.stl" scale="0.001 0.001 0.001"/>
-      </geometry>
-      <material name="orange"/>
-    </visual>
-    <collision>
-        <origin xyz="0 0 0" rpy="0 0 0" />
-      <geometry>
-        <mesh filename="package://seekur_jr_description/meshes/arm/wrist_roll_n.stl" scale="0.001 0.001 0.001"/>
+      <origin xyz="-0.0322 ${0.4*BASE+wrist_roll_link_y_offset} ${-18.5*BASE+wrist_roll_link_x_offset}" rpy="0 -${PI} ${3*PI/2}" />
+      <geometry>
+        <mesh filename="package://seekur_jr_description/meshes/arm/wrist_roll.stl" scale="0.001 0.001 0.001"/>
+      </geometry>
+      <material name="orange"/>
+    </visual>
+    <collision>
+        <origin xyz="-0.0322 ${0.4*BASE+wrist_roll_link_y_offset} ${-18.5*BASE+wrist_roll_link_x_offset}" rpy="0 -${PI} ${3*PI/2}" />
+      <geometry>
+          <mesh filename="package://seekur_jr_description/meshes/arm/wrist_roll.stl" scale="0.001 0.001 0.001"/>
       </geometry>
     </collision>
@@ -418,6 +437,6 @@
   </link>
   <joint name="gripper_l_finger_joint" type="revolute">
-    <origin xyz="${61*BASE} ${27*BASE} ${3*BASE}" rpy="0 0 0"/>
-    <limit effort="1000.0" lower="-${40*(PI/180)}" upper="${13.5*(PI/180)}" velocity="0.5"/>
+    <origin xyz="${gripper_l_finger_joint_x_offset} 0 -0.0145" rpy="0 ${3*PI/2} ${3*PI/2}"/>
+    <limit effort="1000.0" lower="0.0" upper="${40*(PI/180)}" velocity="0.5"/>
     <axis xyz="0 0 -1"/>
     <parent link="wrist_roll_link"/>
@@ -426,7 +445,7 @@
   <link name="gripper_l_finger_link">
     <visual>
-      <origin xyz="0 0 0" rpy="0 0 0" />
-      <geometry>
-        <mesh filename="package://seekur_jr_description/meshes/arm/left_finger_n.stl" scale="0.001 0.001 0.001"/>
+      <origin xyz="0 0 0" rpy="-${3*PI/2.35} -${PI/2} ${3*PI/2}" />
+      <geometry>
+        <mesh filename="package://seekur_jr_description/meshes/arm/left_finger.stl" scale="0.001 0.001 0.001"/>
       </geometry>
       <material name="brown"/>
@@ -442,16 +461,16 @@
   </link>
    <joint name="gripper_r_finger_joint" type="revolute">
-     <origin xyz="${61*BASE} ${-27*BASE} ${3*BASE}" rpy="0 0 0"/>
-     <limit effort="1000.0" lower="-${40*(PI/180)}" upper="${13.5*(PI/180)}"  velocity="0.5"/>
-     <axis xyz="0 0 1"/>
-     <mimic joint="gripper_l_finger_joint"/>
-     <parent link="wrist_roll_link"/>
-     <child link="gripper_r_finger_link"/>
+    <origin xyz="${gripper_r_finger_joint_x_offset} 0 -0.0145" rpy="0 ${3*PI/2} ${3*PI/2}"/>
+    <limit effort="1000.0" lower="0.0" upper="${40*(PI/180)}" velocity="0.5"/>
+    <axis xyz="0 0 1"/>
+    <mimic joint="gripper_l_finger_joint"/>
+    <parent link="wrist_roll_link"/>
+    <child link="gripper_r_finger_link"/>
   </joint>
   <link name="gripper_r_finger_link">
     <visual>
-      <origin xyz="0 0 0" rpy="0 0 0" />
-      <geometry>
-        <mesh filename="package://seekur_jr_description/meshes/arm/right_finger_n.stl" scale="0.001 0.001 0.001"/>
+      <origin xyz="-0.0355 -0.0415 0" rpy="-${3*PI/1.74} -${PI/2} ${3*PI/2}" />
+      <geometry>
+        <mesh filename="package://seekur_jr_description/meshes/arm/right_finger.stl" scale="0.001 0.001 0.001"/>
       </geometry>
       <material name="brown"/>
